File: PCB/lagom.kicad_sch (KiCad schematic)
At the start: 0 parts

Commit message: Grid started
Parts:
- added D? (x72): D_Small, Keebio-Parts:Diode, symbol Device:D_Small
- added J?: Conn_01x04, Connector_PinSocket_2.54mm:PinSocket_1x04_P2.54mm_Vertical, symbol Connector_Generic:Conn_01x04
- added SW? (x57): KEYSW, Button_Switch_Keyboard:SW_Cherry_MX_1.00u_PCB, symbol keyboard_parts:KEYSW
- added SW? (x2): KEYSW, Button_Switch_Keyboard:SW_Cherry_MX_1.75u_PCB, symbol keyboard_parts:KEYSW
- added SW?: KEYSW, Button_Switch_Keyboard:SW_Cherry_MX_1.50u_Plate, symbol keyboard_parts:KEYSW
- added SW? (x6): KEYSW, Button_Switch_Keyboard:SW_Cherry_MX_1.25u_PCB, symbol keyboard_parts:KEYSW
- added SW?: KEYSW, Button_Switch_Keyboard:SW_Cherry_MX_2.75u_PCB, symbol keyboard_parts:KEYSW
- added SW? (x2): RotaryEncoder_Switch, Keebio-Parts:RotaryEncoder_EC11, symbol Device:RotaryEncoder_Switch
- added SW? (x4): KEYSW, Button_Switch_Keyboard:SW_Cherry_MX_1.50u_PCB, symbol keyboard_parts:KEYSW
- added SW? (x3): KEYSW, Button_Switch_Keyboard:SW_Cherry_MX_2.25u_PCB, symbol keyboard_parts:KEYSW
- added SW?: KEYSW, Button_Switch_Keyboard:SW_Cherry_MX_6.25u_PCB, symbol keyboard_parts:KEYSW
- added SW?: KEYSW, Button_Switch_Keyboard:SW_Cherry_MX_2.00u_PCB, symbol keyboard_parts:KEYSW
- added U? (x2): 74HC138, symbol w_logic:74HC138
- added U?: ProMicro, Keebio-Parts:ArduinoProMicro-ZigZag, symbol keebio:ProMicro
Connections:
- new net: SW?.1, SW?.1, SW?.1, SW?.1, SW?.1 (x8)
- new net: D?.2 (A), SW?.2 (x64)
- new net: SW?.1, SW?.1, SW?.1, SW?.1 (x2)
- new net: SW?.1, SW?.1, SW?.1, SW?.1, SW?.1, SW?.1, SW?.1
- new net: D?.1 (K), D?.1 (K), D?.1 (K), D?.1 (K)
- new net: D?.2 (A), SW?.2, SW?.2 (x6)
- new net: SW?.1, SW?.1, SW?.1, SW?.1, SW?.1, SW?.1 (x2)
- new net GND: J?.1 (Pin_1), SW?.C, SW?.C, U?.23 (GND), U?.3 (GND), U?.4 (GND)
- new net RotA: D?.2 (A), SW?.S1
- new net RotB: SW?.1, SW?.1, SW?.1, SW?.1, SW?.S2
- new net RotC: D?.2 (A), SW?.S1
- new net RotD: SW?.1, SW?.1, SW?.1, SW?.1, SW?.S2
- new net SCL: J?.3 (Pin_3), SW?.B, U?.6 (3/PD0)
- new net SDA: J?.4 (Pin_4), SW?.A, U?.5 (2/PD1)
- new net VCC: J?.2 (Pin_2), U?.21 (VCC)
- new net col0: U?.18 (A1/PF6)
- new net col1: U?.17 (A0/PF7)
- new net col2: U?.16 (15/PB1)
- new net col3: U?.15 (14/PB3)
- new net col4: U?.14 (16/PB2)
- new net col5: U?.13 (10/PB6)
- new net encA: SW?.A, U?.1 (TX0/PD3)
- new net encB: SW?.B, U?.2 (RX1/PD2)
- new net rowA: D?.1 (K), D?.1 (K), D?.1 (K), D?.1 (K), D?.1 (K), D?.1 (K), D?.1 (K), D?.1 (K), D?.1 (K), D?.1 (K), D?.1 (K), D?.1 (K), D?.1 (K), D?.1 (K), D?.1 (K), D?.1 (K), D?.1 (K), D?.1 (K), D?.1 (K), D?.1 (K), D?.1 (K), D?.1 (K), D?.1 (K), D?.1 (K), U?.11 (8/PB4)
- new net rowB: U?.12 (9/PB5)
- new net rowC: D?.1 (K), D?.1 (K), D?.1 (K), D?.1 (K), D?.1 (K), D?.1 (K), D?.1 (K), D?.1 (K), D?.1 (K), D?.1 (K), D?.1 (K), D?.1 (K), D?.1 (K), D?.1 (K), D?.1 (K), U?.7 (4/PD4)
- new net rowD: U?.8 (5/PC6)
- new net rowE: D?.1 (K), D?.1 (K), D?.1 (K), D?.1 (K), D?.1 (K), D?.1 (K), D?.1 (K), D?.1 (K), D?.1 (K), D?.1 (K), D?.1 (K), D?.1 (K), D?.1 (K), D?.1 (K), U?.9 (6/PD7)
- new net rowF: U?.10 (7/PE6)
- new net rowG: D?.1 (K), D?.1 (K), D?.1 (K), D?.1 (K), D?.1 (K), D?.1 (K), D?.1 (K), D?.1 (K), D?.1 (K), D?.1 (K), D?.1 (K), U?.19 (A2/PF5), U?.20 (A3/PF4)
- no-connect marks 0 -> 2
