File: PCB/lagom.kicad_sch (KiCad schematic)
At the start: 165 parts, among them J1 Conn_01x04, J2 Conn_01x03, SW1 KEYSW, SW10 KEYSW, SW11 KEYSW, SW12 KEYSW, SW13 KEYSW, SW14 KEYSW, SW15 KEYSW, SW16 KEYSW, SW17 KEYSW, SW18 KEYSW, SW19 KEYSW, SW2 KEYSW, SW20 KEYSW, SW21 KEYSW, SW22 KEYSW, SW23 KEYSW, SW24 KEYSW, SW25 KEYSW, SW26 KEYSW, SW27 KEYSW, SW28 KEYSW, SW29 KEYSW, SW3 KEYSW, SW30 KEYSW, SW31 KEYSW, SW32 KEYSW, SW33 KEYSW, SW34 KEYSW, SW35 KEYSW, SW36 KEYSW, SW37 KEYSW, SW38 KEYSW, SW39 KEYSW, SW4 KEYSW, SW40 KEYSW, SW41 KEYSW, SW42 KEYSW, SW43 KEYSW, SW44 KEYSW, SW45 KEYSW, SW46 KEYSW, SW47 KEYSW, SW48 KEYSW, SW49 KEYSW, SW5 KEYSW, SW50 KEYSW, SW51 KEYSW, SW52 KEYSW, SW53 KEYSW, SW54 KEYSW, SW55 KEYSW, SW56 KEYSW, SW57 KEYSW, SW58 KEYSW, SW59 KEYSW, SW6 KEYSW, SW60 KEYSW, SW61 KEYSW, SW62 KEYSW, SW63 KEYSW, SW64 KEYSW, SW65 KEYSW, SW66 KEYSW, SW67 KEYSW, SW68 KEYSW, SW69 KEYSW, SW7 KEYSW, SW70 KEYSW, SW71 KEYSW, SW72 KEYSW, SW73 KEYSW, SW74 KEYSW, SW75 KEYSW, SW76 KEYSW, SW77 KEYSW, SW78 KEYSW, SW79 KEYSW, SW8 KEYSW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

Commit message: Labelling mostly done
Parts:
- added SW_ENC1, SW_ENC2: KEYSW, Button_Switch_Keyboard:SW_Cherry_MX_1.00u_PCB, symbol keyboard_parts:KEYSW
- D1: footprint Diode_THT:D_DO-35_SOD27_P7.62mm_Horizontal -> Diode_THT:D_DO-34_SOD68_P7.62mm_Horizontal
- SW_ISO_ENT1: renamed from SW33; footprint Button_Switch_Keyboard:SW_Cherry_MX_ISOEnter_PCB -> Button_Switch_Keyboard:SW_Cherry_MX_ISOEnter_PCB_Flipped_Rotated
- SW_STEP_CAPS1: renamed from SW35; footprint Button_Switch_Keyboard:SW_Cherry_MX_1.00u_PCB -> Button_Switch_Keyboard:SW_Cherry_MX_1.25u_PCB
- renumbered SW62 to SW_/1, SW12 to SW_0, SW3 to SW_1, SW4 to SW_2, SW5 to SW_3, SW6 to SW_4, SW7 to SW_5, SW8 to SW_6, SW76 to SW_6.25U_SPACE1, SW9 to SW_7, SW66 to SW_7U_SPACE1, SW10 to SW_8, SW11 to SW_9, SW36 to SW_A1, SW48 to SW_ANSI_ENT1, SW31 to SW_ANSI_\1, SW57 to SW_B1, SW1 to SW_BCKSP1, SW15 to SW_BCKSP_1U1, SW55 to SW_C1, SW34 to SW_CAPS1, SW60 to SW_COMMA1, SW38 to SW_D1, SW16 to SW_DEL1, SW61 to SW_DOT1, SW82 to SW_DOWN1, SW21 to SW_E1, SW32 to SW_END1, SW14 to SW_EQUAL1, SW2 to SW_ESC1, SW39 to SW_F1, SW40 to SW_G1, SW41 to SW_H1, SW17 to SW_HOME1, SW26 to SW_I1, SW51 to SW_ISO_LSHF1, SW47 to SW_ISO_\1, SW52 to SW_ISO_`1, SW42 to SW_J1, SW43 to SW_K1, SW44 to SW_L1, SW69 to SW_LALT_1.25U1, SW73 to SW_LALT_1U1, SW74 to SW_LCMD_1.25U1, SW70 to SW_LCOM_1.5U1, SW68 to SW_LCTRL_1.25U1, SW72 to SW_LCTRL_1.5U1, SW80 to SW_LEFT1, SW50 to SW_LSHF1, SW29 to SW_LSQBR1, SW59 to SW_M1, SW13 to SW_MINUS1, SW58 to SW_N1, SW27 to SW_O1, SW28 to SW_P1, SW65 to SW_PGDN1, SW49 to SW_PGUP1, SW19 to SW_Q1, SW46 to SW_QUOTE1, SW22 to SW_R1, SW81 to SW_RIGHT1, SW63 to SW_RSHIFT1, SW30 to SW_RSQBR1, SW78 to SW_R_CMD1, SW79 to SW_R_CTRL_1.25U1, SW67 to SW_R_CTRL_1.5U1, SW37 to SW_S1, SW45 to SW_SEMICOLON1, SW75 to SW_SPL_SPACE_L1, SW71 to SW_SPL_SPACE_M1, SW77 to SW_SPL_SPACE_R1, SW23 to SW_T1, SW18 to SW_TAB1, SW25 to SW_U1, SW64 to SW_UP1, SW56 to SW_V1, SW20 to SW_W1, SW54 to SW_X1, SW24 to SW_Y1, SW53 to SW_Z1
Connections:
- net LED: now also U1.18 (A1/PF6); no longer U1.7 (4/PD4)
- net RotA: now also SW_ENC1.2
- net RotB: now also SW_ENC1.1, SW_ENC2.1
- net RotC: now also SW_ENC2.2
- net encA: now also U1.7 (4/PD4); no longer U1.18 (A1/PF6)
- net encB: now also U1.8 (5/PC6); no longer U1.17 (A0/PF7)
- net mux0: now also U1.9 (6/PD7); no longer U1.16 (15/PB1)
- net mux1: now also U1.10 (7/PE6); no longer U1.15 (14/PB3)
- net mux2: now also U1.11 (8/PB4); no longer U1.14 (16/PB2)
- net mux3: now also U1.12 (9/PB5); no longer U1.13 (10/PB6)
- net row0: now also U1.13 (10/PB6); no longer U1.12 (9/PB5)
- net row1: now also U1.14 (16/PB2); no longer U1.11 (8/PB4)
- net row2: now also U1.15 (14/PB3); no longer U1.10 (7/PE6)
- net row3: now also U1.16 (15/PB1); no longer U1.9 (6/PD7)
- net row4: now also U1.17 (A0/PF7); no longer U1.8 (5/PC6)

Commit message: Working firmware and updated build guide
Parts:
- added RZ?: RP2040-Zero, symbol rp2040-zero:RP2040-Zero
Connections:
- net LED: now also RZ?.20 (GP29)
- net SCL: now also RZ?.3 (GP2)
- net SDA: now also RZ?.2 (GP1)
- net encA: now also RZ?.4 (GP3)
- net encB: now also RZ?.5 (GP4)
- net mux0: now also RZ?.6 (GP5)
- net mux1: now also RZ?.7 (GP6)
- net mux2: now also RZ?.8 (GP7)
- net mux3: now also RZ?.9 (GP8)
- net row0: now also RZ?.15 (GP14)
- net row1: now also RZ?.16 (GP15)
- net row2: now also RZ?.17 (GP26)
- net row3: now also RZ?.18 (GP27)
- net row4: now also RZ?.19 (GP28)
Changed lines of the file:
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@@
     (effects (font (size 1.27 1.27)) (justify left bottom))
   )
+  (global_label "encD" (shape input) (at 107.569 223.774 0) (fields_autoplaced)
+    (effects (font (size 1.27 1.27)) (justify left))
+    (property "Intersheet References" "${INTERSHEET_REFS}" (id 0) (at 114.5783 223.6946 0)
+      (effects (font (size 1.27 1.27)) (justify left) hide)
+    )
+  )
   (global_label "col6" (shape input) (at 197.104 40.132 90) (fields_autoplaced)
     (effects (font (size 1.27 1.27)) (justify left))
@@
     )
   )
+  (global_label "LED" (shape input) (at 91.44 224.409 0) (fields_autoplaced)
+    (effects (font (size 1.27 1.27)) (justify left))
+    (property "Intersheet References" "${INTERSHEET_REFS}" (id 0) (at 97.3002 224.4884 0)
+      (effects (font (size 1.27 1.27)) (justify left) hide)
+    )
+  )
   (global_label "LED" (shape input) (at 92.329 186.182 0) (fields_autoplaced)
     (effects (font (size 1.27 1.27)) (justify left))
@@
     )
   )
+  (global_label "row4" (shape input) (at 91.44 226.949 0) (fields_autoplaced)
+    (effects (font (size 1.27 1.27)) (justify left))
+    (property "Intersheet References" "${INTERSHEET_REFS}" (id 0) (at 98.3283 227.0284 0)
+      (effects (font (size 1.27 1.27)) (justify left) hide)
+    )
+  )
   (global_label "RotC" (shape input) (at 373.126 88.773 0) (fields_autoplaced)
     (effects (font (size 1.27 1.27)) (justify left))
@@
     )
   )
+  (global_label "row1" (shape input) (at 91.44 234.569 0) (fields_autoplaced)
+    (effects (font (size 1.27 1.27)) (justify left))
+    (property "Intersheet References" "${INTERSHEET_REFS}" (id 0) (at 98.3283 234.6484 0)
+      (effects (font (size 1.27 1.27)) (justify left) hide)
+    )
+  )
   (global_label "col2" (shape input) (at 297.18 177.673 0) (fields_autoplaced)
     (effects (font (size 1.27 1.27)) (justify left))
@@
     )
   )
+  (global_label "mux0" (shape input) (at 62.23 237.109 180) (fields_autoplaced)
+    (effects (font (size 1.27 1.27)) (justify right))
+    (property "Intersheet References" "${INTERSHEET_REFS}" (id 0) (at 54.7369 237.1884 0)
+      (effects (font (size 1.27 1.27)) (justify right) hide)
+    )
+  )
   (global_label "col13" (shape input) (at 356.489 184.912 0) (fields_autoplaced)
     (effects (font (size 1.27 1.27)) (justify left))
@@
     )
   )
+  (global_label "mux1" (shape input) (at 62.23 239.649 180) (fields_autoplaced)
+    (effects (font (size 1.27 1.27)) (justify right))
+    (property "Intersheet References" "${INTERSHEET_REFS}" (id 0) (at 54.7369 239.7284 0)
+      (effects (font (size 1.27 1.27)) (justify right) hide)
+    )
+  )
   (global_label "mux3" (shape input) (at 338.709 184.912 180) (fields_autoplaced)
     (effects (font (size 1.27 1.27)) (justify right))
@@
     )
   )
+  (global_label "encC" (shape input) (at 107.569 221.234 0) (fields_autoplaced)
+    (effects (font (size 1.27 1.27)) (justify left))
+    (property "Intersheet References" "${INTERSHEET_REFS}" (id 0) (at 114.5783 221.1546 0)
+      (effects (font (size 1.27 1.27)) (justify left) hide)
+    )
+  )
+  (global_label "row3" (shape input) (at 91.44 229.489 0) (fields_autoplaced)
+    (effects (font (size 1.27 1.27)) (justify left))
+    (property "Intersheet References" "${INTERSHEET_REFS}" (id 0) (at 98.3283 229.5684 0)
+      (effects (font (size 1.27 1.27)) (justify left) hide)
+    )
+  )
+  (global_label "encB" (shape input) (at 62.23 234.569 180) (fields_autoplaced)
+    (effects (font (size 1.27 1.27)) (justify right))
+    (property "Intersheet References" "${INTERSHEET_REFS}" (id 0) (at 55.2207 234.6484 0)
+      (effects (font (size 1.27 1.27)) (justify right) hide)
+    )
+  )
   (global_label "col12" (shape input) (at 326.136 40.005 90) (fields_autoplaced)
     (effects (font (size 1.27 1.27)) (justify left))
@@
     )
   )
+  (global_label "SDA" (shape input) (at 62.23 226.949 180) (fields_autoplaced)
+    (effects (font (size 1.27 1.27)) (justify right))
+    (property "Intersheet References" "${INTERSHEET_REFS}" (id 0) (at 56.2488 226.8696 0)
+      (effects (font (size 1.27 1.27)) (justify right) hide)
+    )
+  )
   (global_label "row1" (shape input) (at 49.784 74.549 180) (fields_autoplaced)
     (effects (font (size 1.27 1.27)) (justify right))
@@
     )
   )
+  (global_label "row2" (shape input) (at 91.44 232.029 0) (fields_autoplaced)
+    (effects (font (size 1.27 1.27)) (justify left))
+    (property "Intersheet References" "${INTERSHEET_REFS}" (id 0) (at 98.3283 232.1084 0)
+      (effects (font (size 1.27 1.27)) (justify left) hide)
+    )
+  )
   (global_label "row3" (shape input) (at 92.329 191.262 0) (fields_autoplaced)
     (effects (font (size 1.27 1.27)) (justify left))
@@
     )
   )
+  (global_label "SCL" (shape input) (at 62.23 229.489 180) (fields_autoplaced)
+    (effects (font (size 1.27 1.27)) (justify right))
+    (property "Intersheet References" "${INTERSHEET_REFS}" (id 0) (at 56.3093 229.4096 0)
+      (effects (font (size 1.27 1.27)) (justify right) hide)
+    )
+  )
   (global_label "encB" (shape input) (at 56.769 188.722 180) (fields_autoplaced)
     (effects (font (size 1.27 1.27)) (justify right))
@@
     )
   )
+  (global_label "mux2" (shape input) (at 62.23 242.189 180) (fields_autoplaced)
+    (effects (font (size 1.27 1.27)) (justify right))
+    (property "Intersheet References" "${INTERSHEET_REFS}" (id 0) (at 54.7369 242.2684 0)
+      (effects (font (size 1.27 1.27)) (justify right) hide)
+    )
+  )
+  (global_label "encA" (shape input) (at 62.23 232.029 180) (fields_autoplaced)
+    (effects (font (size 1.27 1.27)) (justify right))
+    (property "Intersheet References" "${INTERSHEET_REFS}" (id 0) (at 55.4021 232.1084 0)
+      (effects (font (size 1.27 1.27)) (justify right) hide)
+    )
+  )
   (global_label "col0" (shape input) (at 297.18 172.593 0) (fields_autoplaced)
     (effects (font (size 1.27 1.27)) (justify left))
@@
     )
   )
+  (global_label "row0" (shape input) (at 91.44 237.109 0) (fields_autoplaced)
+    (effects (font (size 1.27 1.27)) (justify left))
+    (property "Intersheet References" "${INTERSHEET_REFS}" (id 0) (at 98.3283 237.1884 0)
+      (effects (font (size 1.27 1.27)) (justify left) hide)
+    )
+  )
   (global_label "col6" (shape input) (at 297.18 187.833 0) (fields_autoplaced)
     (effects (font (size 1.27 1.27)) (justify left))
@@
     )
   )
+  (global_label "mux3" (shape input) (at 62.23 244.729 180) (fields_autoplaced)
+    (effects (font (size 1.27 1.27)) (justify right))
+    (property "Intersheet References" "${INTERSHEET_REFS}" (id 0) (at 54.7369 244.8084 0)
+      (effects (font (size 1.27 1.27)) (justify right) hide)
+    )
+  )
   (symbol (lib_id "keyboard_parts:KEYSW") (at 232.029 88.773 0) (unit 1)
     (in_bom yes) (on_board yes)
@@
     (pin "1")
   )
+  (symbol (lib_id "rp2040-zero:RP2040-Zero") (at 76.2 234.569 0) (unit 1)
+    (in_bom yes) (on_board yes) (fields_autoplaced)
+    (property "Reference" "RZ?" (id 0) (at 78.2194 252.73 0)
+      (effects (font (size 1.27 1.27)) (justify left))
+    )
+    (property "Value" "RP2040-Zero" (id 1) (at 78.2194 255.27 0)
+      (effects (font (size 1.27 1.27)) (justify left))
+    )
+    (property "Footprint" "" (id 2) (at 76.2 234.569 0)
+      (effects (font (size 1.27 1.27)) hide)
+    )
+    (property "Datasheet" "" (id 3) (at 76.2 234.569 0)
+      (effects (font (size 1.27 1.27)) hide)
+    )
+    (pin "1")
+    (pin "10")
+    (pin "11")
+    (pin "12")
+    (pin "13")
+    (pin "14")
+    (pin "15")
+    (pin "16")
+    (pin "17")
+    (pin "18")
+    (pin "19")
+    (pin "2")
+    (pin "20")
+    (pin "21")
+    (pin "22")
+    (pin "23")
+    (pin "3")
+    (pin "4")
+    (pin "5")
+    (pin "6")
+    (pin "7")
+    (pin "8")
+    (pin "9")
+  )
   (symbol (lib_id "keyboard_parts:KEYSW") (at 189.484 68.199 0) (unit 1)
     (in_bom yes) (on_board yes)
@@
       (reference "J2") (unit 1) (value "Conn_01x03") (footprint "Connector_PinSocket_2.54mm:PinSocket_1x03_P2.54mm_Vertical")
     )
+    (path "/2b8cd22b-41b0-4a3f-b88d-8b74deac8136"
+      (reference "RZ?") (unit 1) (value "RP2040-Zero") (footprint "")
+    )
     (path "/7d924492-06b9-4e8b-ad72-2209ecf70752"

Commit message: Build guide updated to show LED socket
Parts:
- removed RZ?: RP2040-Zero, symbol rp2040-zero:RP2040-Zero
Changed lines of the file:
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@@
     (effects (font (size 1.27 1.27)) (justify left bottom))
   )
-  (global_label "encD" (shape input) (at 107.569 223.774 0) (fields_autoplaced)
-    (effects (font (size 1.27 1.27)) (justify left))
-    (property "Intersheet References" "${INTERSHEET_REFS}" (id 0) (at 114.5783 223.6946 0)
-      (effects (font (size 1.27 1.27)) (justify left) hide)
-    )
-  )
   (global_label "col6" (shape input) (at 197.104 40.132 90) (fields_autoplaced)
     (effects (font (size 1.27 1.27)) (justify left))
@@
     )
   )
-  (global_label "LED" (shape input) (at 91.44 224.409 0) (fields_autoplaced)
-    (effects (font (size 1.27 1.27)) (justify left))
-    (property "Intersheet References" "${INTERSHEET_REFS}" (id 0) (at 97.3002 224.4884 0)
-      (effects (font (size 1.27 1.27)) (justify left) hide)
-    )
-  )
   (global_label "LED" (shape input) (at 92.329 186.182 0) (fields_autoplaced)
     (effects (font (size 1.27 1.27)) (justify left))
@@
     )
   )
-  (global_label "row4" (shape input) (at 91.44 226.949 0) (fields_autoplaced)
-    (effects (font (size 1.27 1.27)) (justify left))
-    (property "Intersheet References" "${INTERSHEET_REFS}" (id 0) (at 98.3283 227.0284 0)
-      (effects (font (size 1.27 1.27)) (justify left) hide)
-    )
-  )
   (global_label "RotC" (shape input) (at 373.126 88.773 0) (fields_autoplaced)
     (effects (font (size 1.27 1.27)) (justify left))
@@
     )
   )
-  (global_label "row1" (shape input) (at 91.44 234.569 0) (fields_autoplaced)
-    (effects (font (size 1.27 1.27)) (justify left))
-    (property "Intersheet References" "${INTERSHEET_REFS}" (id 0) (at 98.3283 234.6484 0)
-      (effects (font (size 1.27 1.27)) (justify left) hide)
-    )
-  )
   (global_label "col2" (shape input) (at 297.18 177.673 0) (fields_autoplaced)
     (effects (font (size 1.27 1.27)) (justify left))
@@
     )
   )
-  (global_label "mux0" (shape input) (at 62.23 237.109 180) (fields_autoplaced)
-    (effects (font (size 1.27 1.27)) (justify right))
-    (property "Intersheet References" "${INTERSHEET_REFS}" (id 0) (at 54.7369 237.1884 0)
-      (effects (font (size 1.27 1.27)) (justify right) hide)
-    )
-  )
   (global_label "col13" (shape input) (at 356.489 184.912 0) (fields_autoplaced)
     (effects (font (size 1.27 1.27)) (justify left))
@@
     )
   )
-  (global_label "mux1" (shape input) (at 62.23 239.649 180) (fields_autoplaced)
-    (effects (font (size 1.27 1.27)) (justify right))
-    (property "Intersheet References" "${INTERSHEET_REFS}" (id 0) (at 54.7369 239.7284 0)
-      (effects (font (size 1.27 1.27)) (justify right) hide)
-    )
-  )
   (global_label "mux3" (shape input) (at 338.709 184.912 180) (fields_autoplaced)
     (effects (font (size 1.27 1.27)) (justify right))
@@
     )
   )
-  (global_label "encC" (shape input) (at 107.569 221.234 0) (fields_autoplaced)
-    (effects (font (size 1.27 1.27)) (justify left))
-    (property "Intersheet References" "${INTERSHEET_REFS}" (id 0) (at 114.5783 221.1546 0)
-      (effects (font (size 1.27 1.27)) (justify left) hide)
-    )
-  )
-  (global_label "row3" (shape input) (at 91.44 229.489 0) (fields_autoplaced)
-    (effects (font (size 1.27 1.27)) (justify left))
-    (property "Intersheet References" "${INTERSHEET_REFS}" (id 0) (at 98.3283 229.5684 0)
-      (effects (font (size 1.27 1.27)) (justify left) hide)
-    )
-  )
-  (global_label "encB" (shape input) (at 62.23 234.569 180) (fields_autoplaced)
-    (effects (font (size 1.27 1.27)) (justify right))
-    (property "Intersheet References" "${INTERSHEET_REFS}" (id 0) (at 55.2207 234.6484 0)
-      (effects (font (size 1.27 1.27)) (justify right) hide)
-    )
-  )
   (global_label "col12" (shape input) (at 326.136 40.005 90) (fields_autoplaced)
     (effects (font (size 1.27 1.27)) (justify left))
@@
     )
   )
-  (global_label "SDA" (shape input) (at 62.23 226.949 180) (fields_autoplaced)
-    (effects (font (size 1.27 1.27)) (justify right))
-    (property "Intersheet References" "${INTERSHEET_REFS}" (id 0) (at 56.2488 226.8696 0)
-      (effects (font (size 1.27 1.27)) (justify right) hide)
-    )
-  )
   (global_label "row1" (shape input) (at 49.784 74.549 180) (fields_autoplaced)
     (effects (font (size 1.27 1.27)) (justify right))
@@
     )
   )
-  (global_label "row2" (shape input) (at 91.44 232.029 0) (fields_autoplaced)
-    (effects (font (size 1.27 1.27)) (justify left))
-    (property "Intersheet References" "${INTERSHEET_REFS}" (id 0) (at 98.3283 232.1084 0)
-      (effects (font (size 1.27 1.27)) (justify left) hide)
-    )
-  )
   (global_label "row3" (shape input) (at 92.329 191.262 0) (fields_autoplaced)
     (effects (font (size 1.27 1.27)) (justify left))
@@
     )
   )
-  (global_label "SCL" (shape input) (at 62.23 229.489 180) (fields_autoplaced)
-    (effects (font (size 1.27 1.27)) (justify right))
-    (property "Intersheet References" "${INTERSHEET_REFS}" (id 0) (at 56.3093 229.4096 0)
-      (effects (font (size 1.27 1.27)) (justify right) hide)
-    )
-  )
   (global_label "encB" (shape input) (at 56.769 188.722 180) (fields_autoplaced)
     (effects (font (size 1.27 1.27)) (justify right))
@@
     )
   )
-  (global_label "mux2" (shape input) (at 62.23 242.189 180) (fields_autoplaced)
-    (effects (font (size 1.27 1.27)) (justify right))
-    (property "Intersheet References" "${INTERSHEET_REFS}" (id 0) (at 54.7369 242.2684 0)
-      (effects (font (size 1.27 1.27)) (justify right) hide)
-    )
-  )
-  (global_label "encA" (shape input) (at 62.23 232.029 180) (fields_autoplaced)
-    (effects (font (size 1.27 1.27)) (justify right))
-    (property "Intersheet References" "${INTERSHEET_REFS}" (id 0) (at 55.4021 232.1084 0)
-      (effects (font (size 1.27 1.27)) (justify right) hide)
-    )
-  )
   (global_label "col0" (shape input) (at 297.18 172.593 0) (fields_autoplaced)
     (effects (font (size 1.27 1.27)) (justify left))
@@
     )
   )
-  (global_label "row0" (shape input) (at 91.44 237.109 0) (fields_autoplaced)
-    (effects (font (size 1.27 1.27)) (justify left))
-    (property "Intersheet References" "${INTERSHEET_REFS}" (id 0) (at 98.3283 237.1884 0)
-      (effects (font (size 1.27 1.27)) (justify left) hide)
-    )
-  )
   (global_label "col6" (shape input) (at 297.18 187.833 0) (fields_autoplaced)
     (effects (font (size 1.27 1.27)) (justify left))
@@
     )
   )
-  (global_label "mux3" (shape input) (at 62.23 244.729 180) (fields_autoplaced)
-    (effects (font (size 1.27 1.27)) (justify right))
-    (property "Intersheet References" "${INTERSHEET_REFS}" (id 0) (at 54.7369 244.8084 0)
-      (effects (font (size 1.27 1.27)) (justify right) hide)
-    )
-  )
   (symbol (lib_id "keyboard_parts:KEYSW") (at 232.029 88.773 0) (unit 1)
     (in_bom yes) (on_board yes)
@@
     (pin "1")
   )
-  (symbol (lib_id "rp2040-zero:RP2040-Zero") (at 76.2 234.569 0) (unit 1)
-    (in_bom yes) (on_board yes) (fields_autoplaced)
-    (property "Reference" "RZ?" (id 0) (at 78.2194 252.73 0)
-      (effects (font (size 1.27 1.27)) (justify left))
-    )
-    (property "Value" "RP2040-Zero" (id 1) (at 78.2194 255.27 0)
-      (effects (font (size 1.27 1.27)) (justify left))
-    )
-    (property "Footprint" "" (id 2) (at 76.2 234.569 0)
-      (effects (font (size 1.27 1.27)) hide)
-    )
-    (property "Datasheet" "" (id 3) (at 76.2 234.569 0)
-      (effects (font (size 1.27 1.27)) hide)
-    )
-    (pin "1")
-    (pin "10")
-    (pin "11")
-    (pin "12")
-    (pin "13")
-    (pin "14")
-    (pin "15")
-    (pin "16")
-    (pin "17")
-    (pin "18")
-    (pin "19")
-    (pin "2")
-    (pin "20")
-    (pin "21")
-    (pin "22")
-    (pin "23")
-    (pin "3")
-    (pin "4")
-    (pin "5")
-    (pin "6")
-    (pin "7")
-    (pin "8")
-    (pin "9")
-  )
   (symbol (lib_id "keyboard_parts:KEYSW") (at 189.484 68.199 0) (unit 1)
     (in_bom yes) (on_board yes)
@@
       (reference "J2") (unit 1) (value "Conn_01x03") (footprint "Connector_PinSocket_2.54mm:PinSocket_1x03_P2.54mm_Vertical")
     )
-    (path "/2b8cd22b-41b0-4a3f-b88d-8b74deac8136"
-      (reference "RZ?") (unit 1) (value "RP2040-Zero") (footprint "")
-    )
     (path "/7d924492-06b9-4e8b-ad72-2209ecf70752"
