File: PCB/lagom.kicad_pcb (KiCad board)
At the start: 2 copper layers, 165 parts, among them J1 Conn_01x04, J2 Conn_01x03, SW1 KEYSW, SW10 KEYSW, SW11 KEYSW, SW12 KEYSW, SW13 KEYSW, SW14 KEYSW, SW15 KEYSW, SW16 KEYSW, SW17 KEYSW, SW18 KEYSW, SW19 KEYSW, SW2 KEYSW, SW20 KEYSW, SW21 KEYSW, SW22 KEYSW, SW23 KEYSW, SW24 KEYSW, SW25 KEYSW, SW26 KEYSW, SW27 KEYSW, SW28 KEYSW, SW29 KEYSW, SW3 KEYSW, SW30 KEYSW, SW31 KEYSW, SW32 KEYSW, SW33 KEYSW, SW34 KEYSW, SW35 KEYSW, SW36 KEYSW, SW37 KEYSW, SW38 KEYSW, SW39 KEYSW, SW4 KEYSW, SW40 KEYSW, SW41 KEYSW, SW42 KEYSW, SW43 KEYSW, SW44 KEYSW, SW45 KEYSW, SW46 KEYSW, SW47 KEYSW, SW48 KEYSW, SW49 KEYSW, SW5 KEYSW, SW50 KEYSW, SW51 KEYSW, SW52 KEYSW, SW53 KEYSW, SW54 KEYSW, SW55 KEYSW, SW56 KEYSW, SW57 KEYSW, SW58 KEYSW, SW59 KEYSW, SW6 KEYSW, SW60 KEYSW, SW61 KEYSW, SW62 KEYSW, SW63 KEYSW, SW64 KEYSW, SW65 KEYSW, SW66 KEYSW, SW67 KEYSW, SW68 KEYSW, SW69 KEYSW, SW7 KEYSW, SW70 KEYSW, SW71 KEYSW, SW72 KEYSW, SW73 KEYSW, SW74 KEYSW, SW75 KEYSW, SW76 KEYSW, SW77 KEYSW, SW78 KEYSW, SW79 KEYSW, SW8 KEYSW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

Commit message: Layout and diode placement basically done
Parts:
- D1: footprint Diode_THT:D_DO-35_SOD27_P7.62mm_Horizontal -> Diode_THT:D_DO-34_SOD68_P7.62mm_Horizontal
- D10, D11, D12, D13, D14, D15, D16, D17, D18, D19, D2, D20, D21, D22, D23, D24, D25, D26, D27, D28, D29, D3, D30, D31, D32, D33, D34, D35, D36, D37, D38, D39, D4, D40, D41, D42, D43, D44, D45, D46, D47, D48, D49, D5, D50, D51, D52, D53, D54, D55, D56, D57, D58, D59, D6, D60, D61, D62, D63, D64, D65, D66, D67, D68, D69, D7, D70, D71, D72, D73, D74, D8, D9: footprint Keebio-Parts:Diode -> Diode_THT:D_DO-34_SOD68_P7.62mm_Horizontal
- J2: moved to B.Cu
- SW33: footprint Button_Switch_Keyboard:SW_Cherry_MX_ISOEnter_PCB -> Button_Switch_Keyboard:SW_Cherry_MX_ISOEnter_PCB_Flipped_Rotated
- moved D49 497.7 mm to (245.9, 43.0), turned to -90 degrees
- moved D73 495.5 mm to (272.2, 40.6), turned to -90 degrees
- moved D32 487.7 mm to (288.9, 48.7), turned to -90 degrees
- moved D27 485.1 mm to (234.0, 47.8), turned to -90 degrees
- moved D28 484.1 mm to (241.1, 47.8), turned to -90 degrees
- moved D13 484.0 mm to (260.2, 51.1), turned to -90 degrees
- moved D48 477.9 mm to (291.3, 45.4), turned to -90 degrees
- moved D29 473.6 mm to (257.9, 48.7), turned to -90 degrees
- moved D60 473.2 mm to (207.7, 43.0), turned to -90 degrees
- moved D59 473.1 mm to (202.9, 43.0), turned to -90 degrees
- moved D47 472.6 mm to (279.3, 45.4), turned to -90 degrees
- moved D50 471.7 mm to (253.1, 43.0), turned to -90 degrees
- moved D51 470.7 mm to (269.8, 43.0), turned to -90 degrees
- moved D64 466.9 mm to (117.0, 40.6), turned to -90 degrees
- moved D10 465.5 mm to (217.3, 50.1), turned to -90 degrees
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Connections:
- D13 pad 1: Net-(D13-Pad1) -> row0
- D14 pad 1: Net-(D13-Pad1) -> row0
- D15 pad 1: Net-(D13-Pad1) -> row0
- D16 pad 1: Net-(D13-Pad1) -> row0
- U2 pad 1: mux1 -> mux0
- U2 pad 2: mux2 -> mux1
- U2 pad 3: mux3 -> mux2
- U2 pad 5: mux0 -> mux3
- U3 pad 1: mux1 -> mux0
- U3 pad 2: mux2 -> mux1
- U3 pad 3: mux3 -> mux2
- U3 pad 6: mux0 -> mux3
Other:
- board outline added: 310.4 x 124.2 mm

Commit message: PCB mostly done
Parts:
- SW35: footprint Button_Switch_Keyboard:SW_Cherry_MX_1.00u_PCB -> Button_Switch_Keyboard:SW_Cherry_MX_1.25u_PCB
- moved C2 11.9 mm to (90.7, 40.6)
- moved U3 11.9 mm to (93.8, 46.8)
- moved C1 11.7 mm to (90.7, 52.3)
- moved U2 11.7 mm to (93.8, 58.5)
- moved D29 0.96 mm to (257.9, 47.8)
- moved D30 0.96 mm to (265.0, 47.8)
- moved D31 0.96 mm to (281.7, 47.8)
- moved D32 0.96 mm to (288.9, 47.8)
- moved D13 0.96 mm to (260.2, 50.1)
- moved D14 0.96 mm to (262.6, 50.1)
- moved D15 0.96 mm to (284.1, 50.1)
- moved D16 0.96 mm to (286.5, 50.1)
Connections:
- U1 pad 11: row3 -> row1
- U1 pad 12: row4 -> row0
- U1 pad 17: encD -> encB
- U1 pad 18: encC -> encA
- U1 pad 19: encB -> encD
- U1 pad 20: encA -> encC
- U1 pad 8: row0 -> row4
- U1 pad 9: row1 -> row3
Routing:
- net VCC: track 0.00 -> 383.4 mm
- net col13: track 0.00 -> 318.8 mm
- net col14: track 0.00 -> 318.3 mm
- net col12: track 0.00 -> 300.4 mm
- net RotB: track 0.00 -> 294.1 mm
- net encC: track 0.00 -> 288.1 mm
- net col11: track 0.00 -> 282.5 mm
- net encD: track 0.00 -> 280.4 mm
- net SDA: track 0.00 -> 269.5 mm, vias 0 -> 1
- net SCL: track 0.00 -> 267.4 mm
- net encA: track 0.00 -> 263.2 mm
- net col10: track 0.00 -> 260.3 mm
- net encB: track 0.00 -> 256.8 mm
- net row0: track 0.00 -> 221.8 mm
- net col8: track 0.00 -> 221.4 mm
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Other:
- board size 310.4 x 124.2 mm -> 305.6 x 121.8 mm
