File: PCB/lagom_base/lagom_base.kicad_pcb (KiCad board)
At the start: 2 copper layers, 11 parts

Commit message: V1 done
Parts:
- added G***: LOGO, LOGO, B.Cu at (354.6, 126.5)
- added G***: LOGO, LOGO, B.Cu at (224.4, 126.5)
- added G***: LOGO, LOGO, B.Cu at (94.4, 126.5)
Routing:
- added copper zone on B.Cu, net (none)
- added copper zone on F.Cu, net (none)
Other:
- board outline added: 319.9 x 128.9 mm
- board text added: "JLCJLCJLCJLC"
- board text added: "STHLM KB lagom v1 design by mohoyt"
