File: PCB/lagom_plate/lagom_plate.kicad_pcb (KiCad board)
At the start: 2 copper layers, 319.9 x 128.9 mm, 11 parts

Commit message: Labelling mostly done
Other:
- outline, holes or cut-outs redrawn

Commit message: V1 done
Routing:
- net (no net): vias 0 -> 3
Other:
- board text added: "JLCJLCJLCJLC"
- board text added: "STHLM KB lagom v1 design by mohoyt"
Changed lines of the file:
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@@
       (layerselection 0x00010fc_ffffffff)
       (disableapertmacros false)
-      (usegerberextensions false)
-      (usegerberattributes true)
-      (usegerberadvancedattributes true)
-      (creategerberjobfile true)
+      (usegerberextensions true)
+      (usegerberattributes false)
+      (usegerberadvancedattributes false)
+      (creategerberjobfile false)
       (svguseinch false)
       (svgprecision 6)
@@
       (psa4output false)
       (plotreference true)
-      (plotvalue true)
+      (plotvalue false)
       (plotinvisibletext false)
       (sketchpadsonfab false)
-      (subtractmaskfromsilk false)
+      (subtractmaskfromsilk true)
       (outputformat 1)
       (mirror false)
-      (drillshape 1)
+      (drillshape 0)
       (scaleselection 1)
-      (outputdirectory "")
+      (outputdirectory "gerbers")
     )
   )
@@
   (gr_arc (start 194.05 143.0875) (mid 193.696447 142.941053) (end 193.55 142.5875) (layer "Edge.Cuts") (width 0.05))
   (gr_arc (start 241.8 123.9875) (mid 241.446447 123.841053) (end 241.3 123.4875) (layer "Edge.Cuts") (width 0.05))
+  (gr_text "STHLM KB lagom v1 \ndesign by mohoyt" (at 207.7125 126.5375) (layer "B.SilkS")
+    (effects (font (size 1 1) (thickness 0.15)) (justify mirror))
+  )
+  (gr_text "JLCJLCJLCJLC" (at 329.475 145.6375) (layer "B.SilkS")
+    (effects (font (size 1 1) (thickness 0.15)) (justify mirror))
+  )
+  (via (at 315.15 97.8875) (size 0.8) (drill 0.4) (layers "F.Cu" "B.Cu") (free) (net 0))
+  (via (at 169.5125 155.1875) (size 0.8) (drill 0.4) (layers "F.Cu" "B.Cu") (free) (net 0))
+  (via (at 57.3 102.6625) (size 0.8) (drill 0.4) (layers "F.Cu" "B.Cu") (free) (net 0))
   (group "" (id 02c43930-2c0e-49d9-b811-155189160739)
     (members
